Commit message: Updated name in urdf from visualizer to visualization

File: src/visualization/urdf/pacifica.urdf.xacro (robot description, xacro)
@@ -1,5 +1,4 @@
 <?xml version="1.0"?>
 <robot name="pacifica" xmlns:xacro="http://www.ros.org/wiki/xacro" >
-  <xacro:include filename="$(find visualizer)/urdf/pacifica_18_structure.urdf.xacro" />
-  <!--<xacro:include filename="$(find visualizer)/urdf/example.urdf.xacro" />-->
+  <xacro:include filename="$(find visualization)/urdf/pacifica_18_structure.urdf.xacro" />
 </robot>

File: src/visualization/urdf/pacifica_18_structure.urdf.xacro (robot description, xacro)
@@ -1,5 +1,5 @@
 <?xml version="1.0"?>
 <robot name="pacifica_structure" xmlns:xacro="http://www.ros.org/wiki/xacro" >
-  <xacro:arg name="dae_file" default="$(find visualizer)/meshes/pacifica_18/body.dae"/>
+  <xacro:arg name="dae_file" default="$(find visualization)/meshes/pacifica_18/body.dae"/>
   <xacro:property name="half_track_width" value="0.77" />
   <xacro:property name="half_wheelbase" value="1.54" />
@@ -16,5 +16,5 @@
         <origin xyz="0 0 0" rpy="1.57079632679 ${flip * 3.1415926535} 0" />
         <geometry>
-          <mesh filename="package://visualizer/meshes/pacifica_18/wheel.dae" />
+          <mesh filename="package://visualization/meshes/pacifica_18/wheel.dae" />
         </geometry>
       </visual>
@@ -43,5 +43,5 @@
         <origin xyz="0 0 0" rpy="1.57079632679 ${flip * pi} 0" />
         <geometry>
-          <mesh filename="package://visualizer/meshes/pacifica_18/wheel.dae" />
+          <mesh filename="package://visualization/meshes/pacifica_18/wheel.dae" />
         </geometry>
       </visual>
@@ -90,5 +90,5 @@
       <origin xyz="1.48 0 0.1" rpy="0 0 0" />
       <geometry>
-        <mesh filename="package://visualizer/meshes/pacifica_18/body_collision.stl" scale="0.96 0.96 0.96" />
+        <mesh filename="package://visualization/meshes/pacifica_18/body_collision.stl" scale="0.96 0.96 0.96" />
       </geometry>
       </collision>
